File: HARDWARE_KEYBOARD/kbrd.kicad_sch (KiCad schematic)
At the start: 24 parts, among them J1 USB_C_Receptacle_USB2.0_16P, J2 SWD, SW1 SW_SPST, SW2 SW_SPST, SW3 SW_SPST, SW4 SW_SPST, U1 STM32F103C8Tx, U2 AP2210N-3.3TRG1, Y1 Crystal_GND24

Commit message: Updated PCB & schematic
Parts:
- J2: footprint Connector_PinHeader_2.54mm:PinHeader_1x04_P2.54mm_Vertical -> Connector_PinHeader_2.00mm:PinHeader_1x04_P2.00mm_Vertical
- Y1: footprint Oscillator:Oscillator_SMD_Abracon_ASE-4Pin_3.2x2.5mm -> Oscillator:Oscillator_SMD_Abracon_ASV-4Pin_7.0x5.1mm
Changed lines of the file:
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@@
 			)
 		)
-		(property "Footprint" "Oscillator:Oscillator_SMD_Abracon_ASE-4Pin_3.2x2.5mm"
+		(property "Footprint" "Oscillator:Oscillator_SMD_Abracon_ASV-4Pin_7.0x5.1mm"
 			(at 87.63 107.95 0)
 			(effects
@@
 			)
 		)
-		(property "Footprint" "Connector_PinHeader_2.54mm:PinHeader_1x04_P2.54mm_Vertical"
+		(property "Footprint" "Connector_PinHeader_2.00mm:PinHeader_1x04_P2.00mm_Vertical"
 			(at 198.12 138.43 0)
 			(effects

Commit message: Chane volt regulator footprint to fit the one im going to use
Parts:
- U2: footprint AP2210N-3.3TRG1:SOT95P280X145-3N -> Package_TO_SOT_SMD:SOT-23-3
Changed lines of the file:
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@@
 			)
 		)
-		(property "Footprint" "AP2210N-3.3TRG1:SOT95P280X145-3N"
+		(property "Footprint" "Package_TO_SOT_SMD:SOT-23-3"
 			(at 194.31 58.42 0)
 			(effects
